Commit message: w11

File: src/mecharm_description/urdf/firefighter.urdf.xacro (robot description, xacro)
@@ -11,14 +11,10 @@
     <!-- Import control_xacro -->
     <xacro:include filename="$(find mecharm_moveit_config)/config/firefighter.ros2_control.xacro" />
+    <xacro:firefighter_ros2_control/>
     <!-- <xacro:firefighter_ros2_control
             name="FakeSystem"
             initial_positions_file="$(arg initial_positions_file)"
             use_gazebo="true"/> -->
-    <xacro:firefighter_ros2_control
-            name="$(arg robot_name)"
-            use_gazebo="$(arg use_gazebo)"/>
     <xacro:include filename="$(find mecharm_moveit_config)/config/gazebo_sim_ros2_control.urdf.xacro" />
-    <xacro:load_gazebo_sim_ros2_control_plugin
-      robot_name="$(arg robot_name)"
-      use_gazebo="$(arg use_gazebo)"/>
+    <xacro:load_gazebo_sim_ros2_control_plugin/>
 </robot>

File: src/mecharm_moveit_config/config/firefighter.ros2_control.xacro (robot description, xacro)
@@ -1,69 +1,106 @@
 <?xml version="1.0"?>
 <robot xmlns:xacro="http://www.ros.org/wiki/xacro">
-    <xacro:macro name="firefighter_ros2_control" params="name use_gazebo">
+    <xacro:macro name="firefighter_ros2_control">
         <!-- <xacro:property name="initial_positions" value="${load_yaml(initial_positions_file)['initial_positions']}"/> -->
-        <ros2_control name="${name}" type="system">
+        <ros2_control name="GazeboSimSystem" type="system">
             <hardware>
                 <!-- By default, set up controllers for simulation. This won't work on real hardware -->
-                <xacro:if value="${use_gazebo}">
-                    <plugin>ign_ros2_control/IgnitionSystem</plugin>
-                </xacro:if>
-                <xacro:unless value="${use_gazebo}">
-                  <plugin>mock_components/GenericSystem</plugin>
-                </xacro:unless>
+                    <plugin>gz_ros2_control/GazeboSimSystem</plugin>
             </hardware>
             <joint name="joint1_to_base">
-                <command_interface name="position"/>
-                <command_interface name="velocity"/>
+                <command_interface name="position">
+                  <param name="min">-3.14</param>
+                  <param name="max">3.14</param>
+                </command_interface>
+                <!-- <command_interface name="velocity"/> -->
                 <!-- <state_interface name="position">
                   <param name="initial_value">${initial_positions['joint1_to_base']}</param>
                 </state_interface> -->
                 <state_interface name="velocity"/>
-                <state_interface name="position"/>
+                <state_interface name="position">
+                  <param name="initial_value">0.0</param>
+                </state_interface>
+                <state_interface name="acceleration"/>
+                <state_interface name="effort"/>
             </joint>
             <joint name="joint2_to_joint1">
-                <command_interface name="position"/>
-                <command_interface name="velocity"/>
+                <command_interface name="position">
+                  <param name="min">-3.14</param>
+                  <param name="max">3.14</param>
+                </command_interface>
+                <!-- <command_interface name="velocity"/> -->
                 <!-- <state_interface name="position">
                   <param name="initial_value">${initial_positions['joint2_to_joint1']}</param>
                 </state_interface> -->
                 <state_interface name="velocity"/>
-                <state_interface name="position"/>
+                <state_interface name="position">
+                  <param name="initial_value">0.0</param>
+                </state_interface>
+                <state_interface name="acceleration"/>
+                <state_interface name="effort"/>
             </joint>
             <joint name="joint3_to_joint2">
-                <command_interface name="position"/>
-                <command_interface name="velocity"/>
+                <command_interface name="position">
+                  <param name="min">-3.14</param>
+                  <param name="max">3.14</param>
+                </command_interface>
+                <!-- <command_interface name="velocity"/> -->
                 <!-- <state_interface name="position">
                   <param name="initial_value">${initial_positions['joint3_to_joint2']}</param>
                 </state_interface> -->
                 <state_interface name="velocity"/>
-                <state_interface name="position"/>
+                <state_interface name="position">
+                  <param name="initial_value">0.0</param>
+                </state_interface>
+                <state_interface name="acceleration"/>
+                <state_interface name="effort"/>
             </joint>
             <joint name="joint4_to_joint3">
-                <command_interface name="position"/>
-                <command_interface name="velocity"/>
+                <command_interface name="position">
+                  <param name="min">-3.14</param>
+                  <param name="max">3.14</param>
+                </command_interface>
+                <!-- <command_interface name="velocity"/> -->
                 <!-- <state_interface name="position">
                   <param name="initial_value">${initial_positions['joint4_to_joint3']}</param>
                 </state_interface> -->
                 <state_interface name="velocity"/>
-                <state_interface name="position"/>
+                <state_interface name="position">
+                  <param name="initial_value">0.0</param>
+                </state_interface>
+                <state_interface name="acceleration"/>
+                <state_interface name="effort"/>
             </joint>
             <joint name="joint5_to_joint4">
-                <command_interface name="position"/>
-                <command_interface name="velocity"/>
+                <command_interface name="position">
+                  <param name="min">-3.14</param>
+                  <param name="max">3.14</param>
+                </command_interface>
+                <!-- <command_interface name="velocity"/> -->
                 <!-- <state_interface name="position">
                   <param name="initial_value">${initial_positions['joint5_to_joint4']}</param>
                 </state_interface> -->
                 <state_interface name="velocity"/>
-                <state_interface name="position"/>
+                <state_interface name="position">
+                  <param name="initial_value">0.0</param>
+                </state_interface>
+                <state_interface name="acceleration"/>
+                <state_interface name="effort"/>
             </joint>
             <joint name="joint6_to_joint5">
-                <command_interface name="position"/>
-                <command_interface name="velocity"/>
+                <command_interface name="position">
+                  <param name="min">-3.14</param>
+                  <param name="max">3.14</param>
+                </command_interface>
+                <!-- <command_interface name="velocity"/> -->
                 <!-- <state_interface name="position">
                   <param name="initial_value">${initial_positions['joint6_to_joint5']}</param>
                 </state_interface> -->
                 <state_interface name="velocity"/>
-                <state_interface name="position"/>
+                <state_interface name="position">
+                  <param name="initial_value">0.0</param>
+                </state_interface>
+                <state_interface name="acceleration"/>
+                <state_interface name="effort"/>
             </joint>
         </ros2_control>

File: src/mecharm_moveit_config/config/gazebo_sim_ros2_control.urdf.xacro (robot description, xacro)
@@ -1,15 +1,78 @@
 <?xml version="1.0" ?>
 <robot xmlns:xacro="http://wiki.ros.org/xacro">
-    <xacro:macro name="load_gazebo_sim_ros2_control_plugin" params="robot_name use_gazebo">
-        <xacro:if value="${use_gazebo}">
-            <gazebo>
-                <plugin filename="ign_ros2_control-system" name="ign_ros2_control::IgnitionROS2ControlPlugin">
-                    <parameters>$(find mecharm_moveit_config)/config/ros2_controllers.yaml</parameters>
-                    <ros>
-                        <remapping>/controller_manager/robot_description:=/robot_description</remapping>
-                    </ros>
-                </plugin>
-            </gazebo>
-        </xacro:if>
+    <xacro:macro name="load_gazebo_sim_ros2_control_plugin">
+        <gazebo>
+            <plugin filename="gz_ros2_control-system" name="gz_ros2_control::GazeboSimROS2ControlPlugin">
+                <parameters>$(find mecharm_moveit_config)/config/ros2_controllers.yaml</parameters>
+                <!-- <ros>
+                    <remapping>/controller_manager/robot_description:=/robot_description</remapping>
+                </ros> -->
+                <robot_param>robot_description</robot_param>
+                <robot_param_node>robot_state_publisher</robot_param_node>
+            </plugin>
+        </gazebo>
+          <gazebo reference="base">
+            <visual>
+              <material>
+                <ambient>0 0.8 0 1</ambient>
+                <diffuse>0 0.8 0 1</diffuse>
+                <specular>0 0.8 0 1</specular>
+              </material>
+            </visual>
+          </gazebo>
+          <gazebo reference="link1">
+            <visual>
+              <material>
+                <ambient>0 0 0.8 1</ambient>
+                <diffuse>0 0 0.8 1</diffuse>
+                <specular>0 0 0.8 1</specular>
+              </material>
+            </visual>
+          </gazebo>
+                    <gazebo reference="link2">
+            <visual>
+              <material>
+                <ambient>0 0 0.8 1</ambient>
+                <diffuse>0 0 0.8 1</diffuse>
+                <specular>0 0 0.8 1</specular>
+              </material>
+            </visual>
+          </gazebo>
+                    <gazebo reference="link3">
+            <visual>
+              <material>
+                <ambient>0 0 0.8 1</ambient>
+                <diffuse>0 0 0.8 1</diffuse>
+                <specular>0 0 0.8 1</specular>
+              </material>
+            </visual>
+          </gazebo>
+                    <gazebo reference="link4">
+            <visual>
+              <material>
+                <ambient>0 0 0.8 1</ambient>
+                <diffuse>0 0 0.8 1</diffuse>
+                <specular>0 0 0.8 1</specular>
+              </material>
+            </visual>
+          </gazebo>
+                    <gazebo reference="link5">
+            <visual>
+              <material>
+                <ambient>0 0 0.8 1</ambient>
+                <diffuse>0 0 0.8 1</diffuse>
+                <specular>0 0 0.8 1</specular>
+              </material>
+            </visual>
+          </gazebo>
+                    <gazebo reference="link6">
+            <visual>
+              <material>
+                <ambient>0 0 0.8 1</ambient>
+                <diffuse>0 0 0.8 1</diffuse>
+                <specular>0 0 0.8 1</specular>
+              </material>
+            </visual>
+          </gazebo>
     </xacro:macro>
 </robot>
