Commit message: Extra floating link added, on the floor using urdf file and .dae file

File: src/mecharm_description/urdf/mycobot_280_arm.urdf.xacro (robot description, xacro)
@@ -11,4 +11,5 @@
   <xacro:property name="link5_mass" value="0.11"/>
   <xacro:property name="link6_mass" value="0.0739"/>
+  <xacro:property name="gripper_mass" value="0.12"/>
   <xacro:property name="flange_mass" value="0.035"/>
   <xacro:macro name="link_inertial" params="mass ixx iyy izz">
@@ -124,4 +125,19 @@
       </collision>
     </link>
+        <link name="${prefix}gripper">
+      <xacro:link_inertial mass="${gripper_mass}" ixx="0.00006649" iyy="0.00006649" izz="0.000096"/>
+      <visual>
+        <geometry>
+          <mesh filename="file://$(find mycobot_description)/meshes/mycobot_280/visual/gripper.dae"/>
+        </geometry>
+        <origin xyz="0 0.00 -0.038" rpy="0 0 0"/>
+      </visual>
+      <collision>
+        <geometry>
+          <cylinder radius="0.040" length="0.06"/>
+        </geometry>
+        <origin xyz="0 0.00 0.0" rpy="${-pi/2} 0 0"/>
+      </collision>
+    </link>
     <link name="${prefix}${flange_link}">
       <xacro:link_inertial mass="${flange_mass}" ixx="0.0000149" iyy="0.0000149" izz="0.0000196"/>
@@ -183,4 +199,9 @@
       <origin xyz="0 -0.07318 0" rpy="${pi/2} ${-pi/2} 0"/>
       <dynamics damping="${joint_damping}" friction="${joint_friction}"/>
+    </joint>
+    <joint name="${prefix}link6_to_${prefix}gripper" type="fixed">
+      <parent link="${prefix}$link6"/>
+      <child link="${prefix}gripper"/>
+      <origin xyz="0.05 -0.0318 0" rpy="${pi/2} ${-pi/2} 0"/>
     </joint>
     <joint name="${prefix}link6_to_${prefix}${flange_link}" type="revolute">
@@ -198,4 +219,5 @@
     <xacro:material_visual ref_link="${prefix}link5" ambient="1 1 1 1" diffuse="1 1 1 1" specular="1 1 1 1"/>
     <xacro:material_visual ref_link="${prefix}link6" ambient="1 1 1 1" diffuse="1 1 1 1" specular="1 1 1 1"/>
+    <xacro:material_visual ref_link="${prefix}gripper" ambient="1 1 1 1" diffuse="1 1 1 1" specular="1 1 1 1"/>
     <xacro:material_visual ref_link="${prefix}${flange_link}" ambient="0.5 0.5 0.5 1" diffuse="0.5 0.5 0.5 1" specular="0.5 0.5 0.5 1"/>
   </xacro:macro>
