Commit message: Add forklift model and update physics parameters for improved simulation

File: src/mecharm_description/urdf/mecharm_270_m5.urdf (robot description, URDF)
Before this commit: robot firefighter, 0 links, 0 joints
Links:
- added link fork_horizontal_tine_left; collision box size=0.3 0.05 0.01; visual box size=0.3 0.05 0.01
- added link fork_horizontal_tine_right; collision box size=0.3 0.05 0.01; visual box size=0.3 0.05 0.01
- added link fork_vertical_bar_left; collision box size=0.02 0.02 0.2; visual box size=0.02 0.02 0.2
- added link fork_vertical_bar_right; collision box size=0.02 0.02 0.2; visual box size=0.02 0.02 0.2
- added link forklift_base; collision box size=0.1 0.1 0.02; visual box size=0.1 0.1 0.02
Joints:
- added joint forklift_to_vertical_bar_left: type fixed, parent forklift_base, child fork_vertical_bar_left, origin xyz=0 -0.05 -0.1 rpy=0 0 0
- added joint forklift_to_vertical_bar_right: type fixed, parent forklift_base, child fork_vertical_bar_right, origin xyz=0 0.05 -0.1 rpy=0 0 0
- added joint link6_to_forklift: type fixed, parent link6, child forklift_base, origin xyz=0 0 0 rpy=1.5708 -1.5708 0
- added joint vertical_bar_left_to_tine: type fixed, parent fork_vertical_bar_left, child fork_horizontal_tine_left, origin xyz=0.15 0 -0.1 rpy=0 0 0
- added joint vertical_bar_right_to_tine: type fixed, parent fork_vertical_bar_right, child fork_horizontal_tine_right, origin xyz=0.15 0 -0.1 rpy=0 0 0

Commit message: Update pose of cardboard box in empty world for improved positioning and fix mesh errors to increase RTF

File: src/mecharm_description/urdf/mecharm_270_m5.urdf (robot description, URDF)
Before this commit: robot firefighter, 5 links, 5 joints
Links:
- link fork_horizontal_tine_left: geometry collision box size=0.31 0.055 0.015; visual box size=0.3 0.05 0.01
- link fork_horizontal_tine_right: geometry collision box size=0.31 0.055 0.015; visual box size=0.3 0.05 0.01
- link fork_vertical_bar_left: geometry collision box size=0.025 0.025 0.21; visual box size=0.02 0.02 0.2
- link fork_vertical_bar_right: geometry collision box size=0.025 0.025 0.21; visual box size=0.02 0.02 0.2
- link forklift_base: geometry collision box size=0.12 0.12 0.025; visual box size=0.1 0.1 0.02

Commit message: Adjust dimensions and mass of forklift components; update friction parameters and trajectory timing for improved simulation performance

File: src/mecharm_description/urdf/mecharm_270_m5.urdf (robot description, URDF)
Before this commit: robot firefighter, 5 links, 5 joints
Links:
- link fork_horizontal_tine_left: geometry collision box size=0.225 0.05 0.01; visual box size=0.225 0.05 0.01
- link fork_horizontal_tine_right: geometry collision box size=0.225 0.05 0.01; visual box size=0.225 0.05 0.01
- link fork_vertical_bar_left: geometry collision box size=0.0125 0.0125 0.105; visual box size=0.01 0.01 0.1
- link fork_vertical_bar_right: geometry collision box size=0.0125 0.0125 0.105; visual box size=0.01 0.01 0.1
Joints:
- joint forklift_to_vertical_bar_left: origin xyz=0 -0.05 -0.1 rpy=0 0 0 -> xyz=0 -0.05 -0.05 rpy=0 0 0
- joint forklift_to_vertical_bar_right: origin xyz=0 0.05 -0.1 rpy=0 0 0 -> xyz=0 0.05 -0.05 rpy=0 0 0
- joint vertical_bar_left_to_tine: origin xyz=0.15 0 -0.1 rpy=0 0 0 -> xyz=0.1125 0 -0.05 rpy=0 0 0
- joint vertical_bar_right_to_tine: origin xyz=0.15 0 -0.1 rpy=0 0 0 -> xyz=0.1125 0 -0.05 rpy=0 0 0

Commit message: Refine collision geometry and friction parameters; update cardboard box scale and pose for improved simulation accuracy

File: src/mecharm_description/urdf/mecharm_270_m5.urdf (robot description, URDF)
Before this commit: robot firefighter, 5 links, 5 joints
Links:
- link fork_horizontal_tine_left: geometry collision box size=0.23 0.06 0.015; visual box size=0.225 0.05 0.01
- link fork_horizontal_tine_right: geometry collision box size=0.23 0.06 0.015; visual box size=0.225 0.05 0.01
